File: PCB/free_michelle_v1_0/free_michelle_v1_0.kicad_sch (KiCad schematic)
At the start: 2 parts

Commit message: Dodany do schematu element EEPROM 24AA01
Parts:
- removed GPIO_Controller, TFT_Controller: BlackPill_v2.0_F411_grados73, symbol BluePill_Part_Like_SWD_Breakout_STM:BlackPill_v2.0_F411_grados73
- added C1: 100nF, symbol Device:C
- added CR2032: 3V, symbol Device:Battery_Cell
- added D1: TFT_320x240_ILI9341, symbol grad73_library:TFT_320x240_ILI9341
- added GPIO_CONTROLLER, TFT_CONTROLLER: BlackPill_STM32F4x1_grados73, symbol grad73_library:BlackPill_STM32F4x1_grados73
- added R1: 10k, symbol Device:R_Small
- added R2, R3: 4k7, symbol Device:R_Small
- added U?: 24AA01, symbol grad73_library:24AA01
- added U?: DS3231M, Package_SO:SOIC-16W_7.5x10.3mm_P1.27mm, symbol Timer_RTC:DS3231M
Connections:
- net GND: now also C1.2, CR2032.2 (-), D1.2 (GND), U?.10 (GND), U?.11 (GND), U?.12 (GND), U?.13 (GND), U?.4 (VSS), U?.5 (GND), U?.6 (GND), U?.7 (GND), U?.7 (WP), U?.8 (GND), U?.9 (GND)
- new net: GPIO_CONTROLLER.9 (PA3), TFT_CONTROLLER.8 (PA2)
- new net: GPIO_CONTROLLER.8 (PA2), TFT_CONTROLLER.9 (PA3)
- new net: CR2032.1 (+), U?.14 (VBAT)
- new net +3V3: C1.1, D1.1 (VCC), D1.8 (LED), R1.1, R2.2, R3.2, U?.2 (VCC)
- new net DS3231_IRQ_PA4: R1.2, TFT_CONTROLLER.10 (PA4), U?.3 (~{INT}/SQW)
- new net DS3231_RST_PB15: TFT_CONTROLLER.24 (PB15), U?.4 (~{RST})
- new net DS3231_SCL_PB6: R2.1, R3.1, TFT_CONTROLLER.34 (PB6), U?.16 (SCL)
- new net DS3231_SDA_PB7: TFT_CONTROLLER.35 (PB7), U?.15 (SDA)
- new net TFT_CS_PB12: D1.3 (CS), TFT_CONTROLLER.21 (PB12)
- new net TFT_DC_PB14: D1.5 (DC), TFT_CONTROLLER.23 (PB14)
- new net TFT_MISO_PA6: D1.9 (SDO(MISO)), TFT_CONTROLLER.12 (PA6)
- new net TFT_MOSI_PA7: D1.6 (SDI(MOSI)), TFT_CONTROLLER.13 (PA7)
- new net TFT_RST_PB13: D1.4 (RESET), TFT_CONTROLLER.22 (PB13)
- new net TFT_SCK_PA5: D1.7 (SCK), TFT_CONTROLLER.11 (PA5)
- new net T_TFT_CS_PB10: D1.11 (T_CS), TFT_CONTROLLER.17 (PB10)
- new net T_TFT_IRQ_PA9: D1.14 (T_IRQ), TFT_CONTROLLER.26 (PA9)
- new net T_TFT_MISO_PB4: D1.13 (T_DO), TFT_CONTROLLER.32 (PB4)
- new net T_TFT_MOSI_PB5: D1.12 (T_DIN), TFT_CONTROLLER.33 (PB5)
- new net T_TFT_SCK_PB3: D1.10 (T_CLK), TFT_CONTROLLER.31 (PB3)
- no-connect marks 0 -> 4
Other:
- title: free_michelle_v1_0 -> free_michelle
