File: PCB/free_michelle_v1_0/free_michelle_v1_0.kicad_pcb (KiCad board)
At the start: 2 copper layers, 183.9 x 151.3 mm, 105 parts, among them J1 Zworka_TX, J10 ARK, J11 ARK, J12 Zworka_Buzzer, J13 ARK, J14 ARK, J15 Gniazdo 5VP DC 5,5x2,5, J16 Gniazdo 9V DC 5,5x2,5, J2 Zworka_RX, J3 GROVE_SW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

Commit message: Poprawione warstwy z napisami
Other:
- board text added: "JLCJLCJLCJLC"
